File: schematics/air-detector/board1.kicad_sch (KiCad schematic)
At the start: 31 parts, among them J11 MHZ19B, J12 Conn_01x04_Pin, J5 PMS7003, J8 BME280, U11 SGP41, U12 MQ-136, U2 O2A2, U3 LM358ADR, U5 MQ-7

Commit message: 1. changes in o2a2 sensor; 2. prepare code for o2a2 sensor
Parts:
- R15: value 10K -> 1K
- R15: value 30K -> 330K
- U3: value LM358ADR -> AD8629ARZ
